Commit message: Add arc-clean; smoke test refuses to run with stale nodes

File: arc_description/urdf/arc_bot.urdf.xacro (robot description, xacro)
@@ -102,5 +102,12 @@
   <link name="laser_link">
     <visual><geometry><cylinder radius="0.035" length="0.04"/></geometry></visual>
-    <collision><geometry><cylinder radius="0.035" length="0.04"/></geometry></collision>
+    <!-- NO collision element, deliberately. The LiDAR sensor origin sits at the
+         centre of this link, so a collision cylinder here is geometry the sensor
+         is standing inside: every ray hits it immediately and the whole scan
+         returns the configured minimum range, 0.12 m, in all 360 directions.
+         In RViz that appears as a tight red ring locked around the robot no
+         matter where it drives.
+         A sensor mount needs a visual so you can see it and an inertial so the
+         solver is happy. It does not need collision. -->
     <inertial>
       <mass value="0.15"/>
@@ -112,5 +119,5 @@
       <parent link="base_link"/>
       <child link="laser_link"/>
-      <origin xyz="0.10 0 ${base_height/2 + 0.02}"/>
+      <origin xyz="0.10 0 ${base_height/2 + 0.06}"/>
     </joint>
   </xacro:unless>
@@ -122,5 +129,5 @@
       <parent link="chassis_link"/>
       <child link="laser_link"/>
-      <origin xyz="0.10 0 ${base_height/2 + 0.02}"/>
+      <origin xyz="0.10 0 ${base_height/2 + 0.06}"/>
     </joint>
   </xacro:if>

Commit message: Add arc-clean; smoke test refuses to run with stale nodes

File: arc_description/urdf/arc_bot.urdf.xacro (robot description, xacro)
@@ -101,13 +101,22 @@
        LaserScan message or the costmap will silently receive nothing usable. -->
   <link name="laser_link">
-    <visual><geometry><cylinder radius="0.035" length="0.04"/></geometry></visual>
-    <!-- NO collision element, deliberately. The LiDAR sensor origin sits at the
-         centre of this link, so a collision cylinder here is geometry the sensor
-         is standing inside: every ray hits it immediately and the whole scan
-         returns the configured minimum range, 0.12 m, in all 360 directions.
-         In RViz that appears as a tight red ring locked around the robot no
-         matter where it drives.
-         A sensor mount needs a visual so you can see it and an inertial so the
-         solver is happy. It does not need collision. -->
+    <!-- The visual is offset DOWNWARD so the sensor origin sits above it.
+         gpu_lidar raycasts against the RENDERED scene, which is built from
+         visual geometry rather than collision geometry. A visual centred on the
+         link origin therefore surrounds the sensor, and every one of the 360
+         beams returns the configured minimum range of 0.12 m. The scan is full
+         of plausible numbers at a perfect 10 Hz and the robot is blind; in RViz
+         it shows as a tight red ring that never changes as the robot drives.
+         Removing the COLLISION does not help, which is the trap: collision is
+         what a CPU raycast sensor would use.
+         Housing spans 0.175 to 0.205 m above ground, beam plane at 0.230 m,
+         so there is 0.025 m of clearance. -->
+    <visual>
+      <origin xyz="0 0 -0.04"/>
+      <geometry><cylinder radius="0.035" length="0.03"/></geometry>
+      <material name="arc_black"><color rgba="0.1 0.1 0.1 1"/></material>
+    </visual>
+    <!-- No collision element: see the note above. A sensor mount needs neither
+         collision nor a visual at the beam origin. -->
     <inertial>
       <mass value="0.15"/>
